File: tests/kicad5/fail-project/power.sch (KiCad schematic (older format))
At the start: 2 parts, among them P1 CONN_01X02

Commit message: Imported kicad5/fail-project with KiCad 5.1.5
Parts:
- C1: symbol passive:C -> fail-project-rescue:C-passive
- P1: symbol conn:CONN_01X02 -> fail-project-rescue:CONN_01X02-conn
Changed lines of the file:
@@
 EESchema Schematic File Version 4
-LIBS:good-project-cache
-EELAYER 29 0
+EELAYER 30 0
 EELAYER END
 $Descr A4 11693 8268
@@
 $EndDescr
 $Comp
-L conn:CONN_01X02 P1
+L fail-project-rescue:CONN_01X02-conn P1
 U 1 1 5CA714F2
 P 4350 3610
+AR Path="/5CA714F2" Ref="P1"  Part="1"
+AR Path="/5CA71704/5CA714F2" Ref="P1"  Part="1"
 F 0 "P1" H 4267 3335 50  0000 C CNN
 F 1 "CONN_01X02" H 4267 3426 50  0000 C CNN
@@
 	4850 3560 5450 3560
 $Comp
-L passive:C C1
+L fail-project-rescue:C-passive C1
 U 1 1 5CA745A6
 P 5450 3610
