File: tests/kicad5/good-project-true/logic.sch (KiCad schematic (older format))
At the start: 2 parts

Commit message: Imported kicad5/good-project-true with KiCad 5.1.5
Parts:
- C2: symbol passive:C -> good-project-rescue:C-passive
- R1: symbol passive:R -> good-project-rescue:R-passive
Changed lines of the file:
@@
 EESchema Schematic File Version 4
-LIBS:good-project-cache
-EELAYER 29 0
+EELAYER 30 0
 EELAYER END
 $Descr A4 11693 8268
@@
 $EndDescr
 $Comp
-L passive:R R1
+L good-project-rescue:R-passive R1
 U 1 1 5CA75C86
 P 5500 2790
@@
 $EndComp
 $Comp
-L passive:C C2
+L good-project-rescue:C-passive C2
 U 1 1 5CA76352
 P 5700 2860
