File: tests/kicad5/warning-project/logic.sch (KiCad schematic (older format))
At the start: 2 parts

Commit message: Imported kicad5/warning-project with KiCad 5.1.5
Parts:
- C2: symbol passive:C -> warning-project-rescue:C-passive
- R1: symbol passive:R -> warning-project-rescue:R-passive
Changed lines of the file:
@@
 EESchema Schematic File Version 4
-EELAYER 29 0
+EELAYER 30 0
 EELAYER END
 $Descr A4 11693 8268
@@
 $EndDescr
 $Comp
-L passive:R R1
+L warning-project-rescue:R-passive R1
 U 1 1 5CA75C86
 P 5500 2790
@@
 $EndComp
 $Comp
-L passive:C C2
+L warning-project-rescue:C-passive C2
 U 1 1 5CA76352
 P 5700 2860
