File: tests/kicad5/good-project/good-project.kicad_pcb (KiCad board)
At the start: 6 copper layers, 45.7 x 21.6 mm, 4 parts, among them P1 CONN_01X02

Commit message: Modified the "good" DRC test to be good for KiCad 6
Routing:
- net /Power/VCC: track 14.1 -> 157.2 mm
- net GND: track 15.4 -> 158.6 mm
- net (no net): track 132.0 -> 0.00 mm
